File: hardware/3phasehalfbridge/3phasehalfbridge.kicad_sch (KiCad schematic)
At the start: 70 parts

Commit message: create sch
Parts:
- added J4: Conn_01x02, Connector_AMASS:AMASS_XT30PW-M_1x02_P2.50mm_Horizontal, symbol Connector_Generic:Conn_01x02
- C1, C2, C6: renamed from C?; footprint Capacitor_SMD:C_0402_1005Metric -> Capacitor_SMD:C_0805_2012Metric
- C10, C12: renamed from C?; footprint Capacitor_SMD:C_0402_1005Metric -> Capacitor_SMD:C_0603_1608Metric
- C11, C4, C5, C7, C8: renamed from C?; footprint Capacitor_SMD:C_0402_1005Metric -> Capacitor_SMD:CP_Elec_6.3x3.9
- D1: renamed from D?; footprint Diode_THT:D_DO-35_SOD27_P7.62mm_Horizontal -> Diode_SMD:D_SOD-123F
- D2, D4: renamed from D?; footprint (none) -> Diode_SMD:D_SOD-123F
- J1: renamed from J?; footprint (none) -> Connector_PinHeader_2.54mm:PinHeader_1x16_P2.54mm_Vertical
- J2: renamed from J?; footprint (none) -> Connector_Wire:SolderWire-1.5sqmm_1x02_P7.8mm_D1.7mm_OD3.9mm
- J3: renamed from J?; footprint (none) -> Connector_AMASS:AMASS_MR30PW-FB_1x03_P3.50mm_Horizontal
- L1, L2: renamed from L?; footprint (none) -> Inductor_SMD:L_Taiyo-Yuden_MD-5050
- R1, R10, R11, R12, R13, R14, R15, R18, R19, R2, R20, R3, R4, R5, R6, R7, R8, R9: renamed from R?; footprint (none) -> Resistor_SMD:R_0402_1005Metric
- R16, R17: renamed from R?; footprint (none) -> Resistor_SMD:R_2512_6332Metric
- U1: renamed from U?; footprint (none) -> Package_DFN_QFN:DFN-6-1EP_3x2mm_P0.5mm_EP1.65x1.35mm
- U8, U9: renamed from U?; footprint (none) -> Package_SO:MSOP-8_3x3mm_P0.65mm
- gave numbers to parts that had none: 29
Connections:
- net GND: now also J4.1 (Pin_1); no longer C19.2, Q6.1 (S), Q6.2 (S), Q6.3 (S), Q7.5 (D), R16.1, U6.6 (HS), U8.8 (IN+)
- net at C17.2, Q2.1 (S), Q2.2 (S)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: no longer R10.1
- net at U4.7 (HO): now also R10.1
- net VIN: no longer names the net of Q1.1 (S), Q1.2 (S), Q1.3 (S), U1.2 (IN)
- net VIN: now also J4.2 (Pin_2)
- new net: C19.2, Q6.1 (S), Q6.2 (S), Q6.3 (S), Q7.5 (D), R16.1, U6.6 (HS), U8.8 (IN+)
Other:
- moved on the sheet: C1, C10, C11, C12, C13, C2, C3, C4, C5, C6, C7, C8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
